File: electronics/ESP32CAM-Weather-Station/ESP32CAM-Weather-Station.kicad_pcb (KiCad board)
At the start: 4 copper layers, 0 parts

Commit message: [WIP] Added board shape.
Other:
- board outline added: 100 x 100 mm
