File: electronics/ESP32CAM-Weather-Station/ESP32CAM-Weather-Station.kicad_pcb (KiCad board)
At the start: 4 copper layers, 100 x 100 mm, 94 parts, among them IC1 BME688, IC2 SGP41-D-R4, IC3 VEML7700-TT, IC4 BQ24093DGQR, IC5 BQ29707DSET, IC6 MCP3426A0T-E_SN, IC7 TPS63070RNMR, J1 B4B-PH-SM4-TB_LF__SN_, J10 Conn_01x02_Pin, J2 B4B-PH-SM4-TB_LF__SN_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

Commit message: [Self-review] Added via stiching on power supply side ground.
Routing:
- net GND: vias 90 -> 203
